File: hardware/TTExperimentModule/TTExperimentModule.kicad_sch (KiCad schematic)
At the start: 25 parts, among them J1 Conn_01x03, J2 Conn_01x02, J3 5050700622, U1 74CBTLV3257, U2 AP2112K-1.8, U3 AP2112K-3.3

Commit message: BOM updates for spaaaaaace
Parts:
- C1, C5: LCSC C408142 -> (none); MPN GRM21BR71C106KE51L -> (none)
- C2, C6: DigikeyPN (none) -> 587-3410-1-ND; LCSC C5673 -> (none); MPN CL10A105KA8NNNC -> LMK107B7105KAHT
- C3, C7: DigikeyPN (none) -> 490-18203-1-ND; LCSC C100072 -> (none); MPN CL05A104KA5NNNC -> GCM155L81E104KE02D
- C4: DigikeyPN (none) -> 490-18203-1-ND; MPN CL05A104KA5NNNC -> GCM155L81E104KE02D
- FB1, FB2: DigikeyPN (none) -> 490-14032-1-ND; MPN (none) -> BLM18KG601BH1D
- R1, R2, R3, R4, R5: DigikeyPN (none) -> 10-ERJ-H2GJ103XCT-ND; MPN RC0402FR-0710KL -> ERJ-H2GJ103X
- R6: DigikeyPN (none) -> 10-ERJ-H2GJ102XCT-ND; MPN CR0402-FX-1001GLF -> ERJ-H2GJ102X
- U1: DigikeyPN (none) -> 1727-4410-1-ND
